File: simple_led_torch.kicad_sch (KiCad schematic)
At the start: 4 parts, among them SW1 DPST_Push_Button

Commit message: update footprints
Parts:
- B1: footprint (none) -> simple_led_torch:2032_Battery_Holder
- D1: footprint (none) -> simple_led_torch:LED_L10mm_D2.54mm
- R1: footprint (none) -> simple_led_torch:R_Axial_L8mm_D2.5mm_Horizontal
- SW1: footprint (none) -> simple_led_torch:DPST_L6.5mm_D4.5mm
Changed lines of the file:
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@@
   (title_block
     (title "Simple LED Torch")
-    (date "2022-01-27")
-    (rev "V01")
+    (date "2022-01-28")
+    (rev "V02")
     (company "SELF")
     (comment 1 "Author: Sunder")
+    (comment 2 "Added Footprints")
   )
   (polyline (pts (xy 104.14 66.04) (xy 142.24 66.04))
@@
       (effects (font (size 0.5 0.5)))
     )
-    (property "Footprint" "" (id 2) (at 132.588 71.12 0)
+    (property "Footprint" "simple_led_torch:DPST_L6.5mm_D4.5mm" (id 2) (at 132.588 71.12 0)
       (effects (font (size 1.27 1.27)) hide)
     )
@@
       (effects (font (size 0.5 0.5)))
     )
-    (property "Footprint" "" (id 2) (at 111.76 71.12 0)
+    (property "Footprint" "simple_led_torch:LED_L10mm_D2.54mm" (id 2) (at 111.76 71.12 0)
       (effects (font (size 1.27 1.27)) hide)
     )
@@
       (effects (font (size 0.5 0.5)))
     )
-    (property "Footprint" "" (id 2) (at 122.428 78.74 0)
+    (property "Footprint" "simple_led_torch:2032_Battery_Holder" (id 2) (at 122.428 78.74 0)
       (effects (font (size 1.27 1.27)) (justify left) hide)
     )
@@
       (effects (font (size 0.5 0.5)))
     )
-    (property "Footprint" "" (id 2) (at 122.428 71.12 0)
+    (property "Footprint" "simple_led_torch:R_Axial_L8mm_D2.5mm_Horizontal" (id 2) (at 122.428 71.12 0)
       (effects (font (size 1.27 1.27)) (justify left) hide)
     )
@@
   (symbol_instances
     (path "/790ac756-4e5a-4e12-8ad6-660a17d6e2a9"
-      (reference "B1") (unit 1) (value "Battery_Cell") (footprint "")
+      (reference "B1") (unit 1) (value "Battery_Cell") (footprint "simple_led_torch:2032_Battery_Holder")
     )
     (path "/49668e46-eb59-462e-ba8d-d3fa337d03dd"
-      (reference "D1") (unit 1) (value "Led") (footprint "")
+      (reference "D1") (unit 1) (value "Led") (footprint "simple_led_torch:LED_L10mm_D2.54mm")
     )
     (path "/be08841c-2284-4665-8490-171bc25e29f4"
-      (reference "R1") (unit 1) (value "330") (footprint "")
+      (reference "R1") (unit 1) (value "330") (footprint "simple_led_torch:R_Axial_L8mm_D2.5mm_Horizontal")
     )
     (path "/3709e52a-85ad-4022-9dd6-3aa933a394cd"
-      (reference "SW1") (unit 1) (value "DPST_Push_Button") (footprint "")
+      (reference "SW1") (unit 1) (value "DPST_Push_Button") (footprint "simple_led_torch:DPST_L6.5mm_D4.5mm")
     )
   )

Commit message: done
Parts:
- added unit 2 of SW1
Connections:
- no-connect marks 0 -> 2
Other:
- note added: "No Connect"
Changed lines of the file:
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@@
     (company "SELF")
     (comment 1 "Author: Sunder")
-    (comment 2 "Added Footprints")
-  )
+    (comment 5 "Added Footprints")
+  )
+  (no_connect (at 156.21 77.47))
+  (no_connect (at 148.59 77.47))
   (polyline (pts (xy 104.14 66.04) (xy 142.24 66.04))
     (stroke (width 0) (type default) (color 0 0 0 0))
   )
+  (polyline (pts (xy 162.56 66.04) (xy 162.56 83.82))
+    (stroke (width 0) (type default) (color 0 0 0 0))
+  )
+  (polyline (pts (xy 162.56 83.82) (xy 142.24 83.82))
+    (stroke (width 0) (type default) (color 0 0 0 0))
+  )
   (wire (pts (xy 109.22 71.12) (xy 106.68 71.12))
     (stroke (width 0) (type default) (color 0 0 0 0))
@@
     (stroke (width 0) (type default) (color 0 0 0 0))
   )
+  (polyline (pts (xy 142.24 66.04) (xy 162.56 66.04))
+    (stroke (width 0) (type default) (color 0 0 0 0))
+  )
   (wire (pts (xy 126.238 71.12) (xy 128.778 71.12))
     (stroke (width 0) (type default) (color 0 0 0 0))
@@
   (wire (pts (xy 106.68 78.74) (xy 119.634 78.74))
     (stroke (width 0) (type default) (color 0 0 0 0))
+  )
+  (text "No Connect" (at 148.59 68.58 0)
+    (effects (font (size 0.8 0.8) (thickness 0.254) bold italic) (justify left bottom))
   )
   (text "Simple LED Torch" (at 114.3 66.04 0)
     (effects (font (size 1.27 1.27) (thickness 0.254) bold italic) (justify left bottom))
   )
+  (symbol (lib_id "Lion_Logo:LOGO") (at 204.47 176.53 0) (mirror y) (unit 1)
+    (in_bom yes) (on_board yes) (fields_autoplaced)
+    (property "Reference" "#G1" (id 0) (at 204.47 167.7808 0)
+      (effects (font (size 1.27 1.27)) hide)
+    )
+    (property "Value" "LOGO" (id 1) (at 204.47 185.2792 0)
+      (effects (font (size 1.27 1.27)) hide)
+    )
+    (property "Footprint" "" (id 2) (at 204.47 176.53 0)
+      (effects (font (size 1.27 1.27)) hide)
+    )
+    (property "Datasheet" "" (id 3) (at 204.47 176.53 0)
+      (effects (font (size 1.27 1.27)) hide)
+    )
+  )
   (symbol (lib_id "simple_led_torch:DPST_Push_Button") (at 132.588 71.12 0) (unit 1)
     (in_bom yes) (on_board yes)
@@
     (pin "2")
   )
+  (symbol (lib_id "simple_led_torch:DPST_Push_Button") (at 152.4 77.47 0) (unit 2)
+    (in_bom yes) (on_board yes) (fields_autoplaced)
+    (property "Reference" "SW1" (id 0) (at 152.4 71.12 0))
+    (property "Value" "DPST_Push_Button" (id 1) (at 152.4 73.66 0))
+    (property "Footprint" "simple_led_torch:DPST_L6.5mm_D4.5mm" (id 2) (at 152.4 89.662 0)
+      (effects (font (size 1.27 1.27)) (justify left) hide)
+    )
+    (property "Datasheet" "https://www.mouser.in/datasheet/2/670/ts02-2586188.pdf" (id 3) (at 152.4 81.534 0)
+      (effects (font (size 1.27 1.27)) (justify left) hide)
+    )
+    (property "Purchase Link" "https://www.mouser.in/ProductDetail/CUI-Devices/TS02-66-110-BK-160-SCR-D?qs=A6eO%252BMLsxmQ7CWdunsyhcQ%3D%3D" (id 4) (at 152.4 83.566 0)
+      (effects (font (size 1.27 1.27)) (justify left) hide)
+    )
+    (property "Vender" "Mouser" (id 5) (at 152.4 85.598 0)
+      (effects (font (size 1.27 1.27)) (justify left) hide)
+    )
+    (property "Part Number" "179-TS0266110BK160SC" (id 6) (at 152.4 87.884 0)
+      (effects (font (size 1.27 1.27)) (justify left) hide)
+    )
+    (pin "3")
+    (pin "4")
+  )
   (symbol (lib_id "simple_led_torch:Battery_Cell") (at 122.428 78.74 0) (mirror y) (unit 1)
     (in_bom yes) (on_board yes)
@@
   )
   (symbol_instances
+    (path "/2f3ca0b5-8e5a-4cbf-b14b-e359ff3d88c2"
+      (reference "#G1") (unit 1) (value "LOGO") (footprint "")
+    )
     (path "/790ac756-4e5a-4e12-8ad6-660a17d6e2a9"
       (reference "B1") (unit 1) (value "Battery_Cell") (footprint "simple_led_torch:2032_Battery_Holder")
@@
       (reference "SW1") (unit 1) (value "DPST_Push_Button") (footprint "simple_led_torch:DPST_L6.5mm_D4.5mm")
     )
-  )
+    (path "/61904185-9b01-4148-bd41-e6cfbcfdd06f"
+      (reference "SW1") (unit 2) (value "DPST_Push_Button") (footprint "simple_led_torch:DPST_L6.5mm_D4.5mm")
+    )
+  )
